Commit message: added gazebo files

File: description/robot.urdf.xacro (robot description, xacro)
@@ -2,3 +2,4 @@
 <robot xmlns:xacro="http://www.ros.org/wiki/xacro" name="auriga" >
     <xacro:include filename="robot_core.xacro" />
+    <!-- <xacro:include filename="gazebo_control.xacro" /> -->
 </robot>

File: description/robot_core.xacro (robot description, xacro)
@@ -20,5 +20,5 @@
      <child link="base_link"/>
    </joint>
-    <link
+ <link
     name="base_link">
     <inertial>
@@ -64,15 +64,15 @@
     <inertial>
       <origin
-        xyz="-0.0031943 0.077406 0.051422"
-        rpy="0 0 0" />
-      <mass
-        value="1.4" />
-      <inertia
-        ixx="0.0029865"
-        ixy="1.1235E-05"
-        ixz="3.1664E-05"
-        iyy="0.0025991"
-        iyz="-0.00067818"
-        izz="0.00041191" />
+        xyz="-0.00319427397416952 0.0774063348676216 0.0514223730363776"
+        rpy="0 0 0" />
+      <mass
+        value="0.157115010617485" />
+      <inertia
+        ixx="0.0029864627992537"
+        ixy="1.12349826817264E-05"
+        ixz="3.1664433625397E-05"
+        iyy="0.00259908313149434"
+        iyz="-0.000678181482698449"
+        izz="0.000411909267858246" />
     </inertial>
     <visual>
@@ -87,5 +87,5 @@
         name="">
         <color
-          rgba="0.42745 0.44706 0.42745 1" />
+          rgba="0.427450980392157 0.447058823529412 0.427450980392157 1" />
       </material>
     </visual>
@@ -117,15 +117,15 @@
     <inertial>
       <origin
-        xyz="0.0023959 -0.061899 -8.3267E-17"
-        rpy="0 0 0" />
-      <mass
-        value="1" />
+        xyz="0.0023959 -0.061899 -0.00023965"
+        rpy="0 0 0" />
+      <mass
+        value="0.109" />
       <inertia
         ixx="0.00075509"
-        ixy="4.3843E-06"
-        ixz="7.2993E-20"
-        iyy="0.00066526"
-        iyz="-3.1639E-20"
-        izz="0.0001028" />
+        ixy="4.3842E-06"
+        ixz="1.6974E-08"
+        iyy="0.00066525"
+        iyz="2.1776E-06"
+        izz="0.00010281" />
     </inertial>
     <visual>
@@ -157,5 +157,5 @@
     type="revolute">
     <origin
-      xyz="-0.02051 0.053967 -0.1"
+      xyz="-0.02051 0.053967 -0.099947"
       rpy="0 0 3.1416" />
     <parent
@@ -175,15 +175,15 @@
     <inertial>
       <origin
-        xyz="0.0073954 -0.00033419 5.8975E-05"
-        rpy="0 0 0" />
-      <mass
-        value="1.3" />
-      <inertia
-        ixx="0.0022259"
-        ixy="4.5416E-06"
-        ixz="-8.1867E-07"
-        iyy="0.0014255"
-        iyz="8.9816E-07"
-        izz="0.0014302" />
+        xyz="0.00416147173779097 -9.28831021262955E-08 1.94176211321812E-07"
+        rpy="0 0 0" />
+      <mass
+        value="0.926156136524473" />
+      <inertia
+        ixx="0.00219829054546711"
+        ixy="-1.07358910102717E-08"
+        ixz="8.07356099787813E-09"
+        iyy="0.00140016164031924"
+        iyz="3.89529542945175E-08"
+        izz="0.00140018200801187" />
     </inertial>
     <visual>
@@ -198,5 +198,5 @@
         name="">
         <color
-          rgba="0.75294 0.75294 0.75294 1" />
+          rgba="0.752941176470588 0.752941176470588 0.752941176470588 1" />
       </material>
     </visual>
@@ -215,6 +215,6 @@
     type="continuous">
     <origin
-      xyz="0.0906500000000005 -0.0786880243269096 0.0900000000000002"
-      rpy="0 0 3.14159265358979" />
+      xyz="0.10265 -0.079036 0.089695"
+      rpy="0 0 3.1416" />
     <parent
       link="bogie_1_link" />
@@ -228,15 +228,15 @@
     <inertial>
       <origin
-        xyz="0.0073954 -0.0003392 -0.38999"
-        rpy="0 0 0" />
-      <mass
-        value="1.3" />
-      <inertia
-        ixx="0.0022259"
-        ixy="4.6122E-06"
-        ixz="-1.5572E-07"
-        iyy="0.0014254"
-        iyz="1.9352E-07"
-        izz="0.0014304" />
+        xyz="0.0041615 -0.00034885 -0.39025"
+        rpy="0 0 0" />
+      <mass
+        value="0.92616" />
+      <inertia
+        ixx="0.0021983"
+        ixy="9.9644E-09"
+        ixz="-9.0085E-09"
+        iyy="0.0014002"
+        iyz="4.0148E-08"
+        izz="0.0014002" />
     </inertial>
     <visual>
@@ -268,6 +268,6 @@
     type="continuous">
     <origin
-      xyz="0.09065 -0.0786880243269102 0.3"
-      rpy="0 0 3.14159265358979" />
+      xyz="0.10265 -0.078688 0.29995"
+      rpy="0 0 3.1416" />
     <parent
       link="bogie_1_link" />
@@ -281,15 +281,15 @@
     <inertial>
       <origin
-        xyz="0.0073954 0.00024372 0.39024"
-        rpy="0 0 0" />
-      <mass
-        value="1.3" />
-      <inertia
-        ixx="0.0022259"
-        ixy="-3.3261E-06"
-        ixz="-3.199E-06"
-        iyy="0.0014277"
-        iyz="-2.5036E-06"
-        izz="0.001428" />
+        xyz="0.00416147173779091 0.000348722601230034 0.39025104440836"
+        rpy="0 0 0" />
+      <mass
+        value="0.926156136524472" />
+      <inertia
+        ixx="0.00219829054546711"
+        ixy="-1.32650632923669E-08"
+        ixz="-2.11656297334914E-09"
+        iyy="0.00140013325413858"
+        iyz="-1.15497356200624E-08"
+        izz="0.00140021039419254" />
     </inertial>
     <visual>
@@ -304,5 +304,5 @@
         name="">
         <color
-          rgba="0.75294 0.75294 0.75294 1" />
+          rgba="0.752941176470588 0.752941176470588 0.752941176470588 1" />
       </material>
     </visual>
@@ -321,5 +321,5 @@
     type="continuous">
     <origin
-      xyz="-0.111159632502295 0.132654956914557 -0.19"
+      xyz="-0.12316 0.13231 -0.19025"
       rpy="0 0 0" />
     <parent
@@ -337,5 +337,5 @@
         rpy="0 0 0" />
       <mass
-        value="1.4" />
+        value="0.15712" />
       <inertia
         ixx="0.0029865"
@@ -387,15 +387,15 @@
     <inertial>
       <origin
-        xyz="0.0023959 0.061897 -0.00066505"
-        rpy="0 0 0" />
-      <mass
-        value="1" />
-      <inertia
-        ixx="0.00075509"
-        ixy="-4.384E-06"
-        ixz="4.7104E-08"
-        iyy="0.00066519"
-        iyz="-6.0427E-06"
-        izz="0.00010286" />
+        xyz="0.00239591308301151 0.0617953988436242 0.00358741675136703"
+        rpy="0 0 0" />
+      <mass
+        value="0.108995977851336" />
+      <inertia
+        ixx="0.0007550940265459"
+        ixy="-4.37688335423889E-06"
+        ixz="-2.54091808736551E-07"
+        iyy="0.000663370668469634"
+        iyz="3.25430149906427E-05"
+        izz="0.000104686998401709" />
     </inertial>
     <visual>
@@ -410,5 +410,5 @@
         name="">
         <color
-          rgba="0.42745 0.44706 0.42745 1" />
+          rgba="0.427450980392157 0.447058823529412 0.427450980392157 1" />
       </material>
     </visual>
@@ -427,5 +427,5 @@
     type="revolute">
     <origin
-      xyz="-0.32665 -0.038688 0.066853"
+      xyz="-0.32665 -0.038665 0.067793"
       rpy="3.1416 0 3.1416" />
     <parent
@@ -445,15 +445,15 @@
     <inertial>
       <origin
-        xyz="6.7458E-05 -0.00033338 -0.0073954"
-        rpy="0 0 0" />
-      <mass
-        value="1.3" />
-      <inertia
-        ixx="0.0014302"
-        ixy="1.016E-06"
-        ixz="9.3391E-07"
-        iyy="0.0014256"
-        iyz="-4.5193E-06"
-        izz="0.0022259" />
+        xyz="-2.1518E-07 -5.3832E-09 -0.0041615"
+        rpy="0 0 0" />
+      <mass
+        value="0.92616" />
+      <inertia
+        ixx="0.0014001"
+        ixy="3.1138E-08"
+        ixz="1.2067E-08"
+        iyy="0.0014002"
+        iyz="-5.9011E-09"
+        izz="0.0021983" />
     </inertial>
     <visual>
@@ -485,6 +485,6 @@
     type="continuous">
     <origin
-      xyz="0.0906500000000001 0.0796504434421384 0.0891493804349932"
-      rpy="0 -1.5707963267949 0" />
+      xyz="0.10265 0.07334 0.094409"
+      rpy="0 1.5708 0" />
     <parent
       link="bogie_2_link" />
@@ -498,15 +498,15 @@
     <inertial>
       <origin
-        xyz="-0.0073954 0.00028789 -0.00018094"
-        rpy="0 0 0" />
-      <mass
-        value="1.3" />
-      <inertia
-        ixx="0.0022259"
-        ixy="3.9131E-06"
-        ixz="-2.4463E-06"
-        iyy="0.0014267"
-        iyz="2.2425E-06"
-        izz="0.001429" />
+        xyz="-0.0041615 -2.0875E-07 5.2503E-08"
+        rpy="0 0 0" />
+      <mass
+        value="0.92616" />
+      <inertia
+        ixx="0.0021983"
+        ixy="1.0043E-08"
+        ixz="-8.9202E-09"
+        iyy="0.0014002"
+        iyz="3.9846E-08"
+        izz="0.0014002" />
     </inertial>
     <visual>
@@ -538,5 +538,5 @@
     type="continuous">
     <origin
-      xyz="0.09065 0.0777165216962496 -0.0908402302281802"
+      xyz="0.10265 0.0837717629834123 -0.0852883163107575"
       rpy="0 0 0" />
     <parent
@@ -551,15 +551,15 @@
     <inertial>
       <origin
-        xyz="-0.0073954 0.00030624 0.00014786"
-        rpy="0 0 0" />
-      <mass
-        value="1.3" />
-      <inertia
-        ixx="0.0022259"
-        ixy="4.1463E-06"
-        ixz="2.0259E-06"
-        iyy="0.0014263"
-        iyz="-1.9924E-06"
-        izz="0.0014294" />
+        xyz="-0.00416147173779097 -6.99332501352679E-08 2.03570656609475E-07"
+        rpy="0 0 0" />
+      <mass
+        value="0.926156136524472" />
+      <inertia
+        ixx="0.0021982905454671"
+        ixy="-1.99317804403964E-09"
+        ixz="-1.32841629112928E-08"
+        iyy="0.00140021060221958"
+        iyz="-1.08307848249764E-08"
+        izz="0.00140013304611153" />
     </inertial>
     <visual>
@@ -574,5 +574,5 @@
         name="">
         <color
-          rgba="0.75294 0.75294 0.75294 1" />
+          rgba="0.752941176470588 0.752941176470588 0.752941176470588 1" />
       </material>
     </visual>
@@ -591,6 +591,6 @@
     type="continuous">
     <origin
-      xyz="-0.417304617315038 0.0399992013357422 -0.2329999973597"
-      rpy="3.14159265358979 0 3.14159265358979" />
+      xyz="-0.4293 0.04 -0.233"
+      rpy="3.1416 0 3.1416" />
     <parent
       link="rocker_2_link" />
@@ -604,15 +604,15 @@
     <inertial>
       <origin
-        xyz="0.022525 0.025224 0.0068988"
-        rpy="0 0 0" />
-      <mass
-        value="0.1" />
-      <inertia
-        ixx="4.4351E-05"
-        ixy="2.9037E-08"
-        ixz="-1.5175E-07"
-        iyy="6.9475E-05"
-        iyz="3.35E-07"
-        izz="2.791E-05" />
+        xyz="0.0225246315179786 0.0252244678162723 0.00689883757739537"
+        rpy="0 0 0" />
+      <mass
+        value="0.0941041855286772" />
+      <inertia
+        ixx="4.43514677561826E-05"
+        ixy="2.9036632805171E-08"
+        ixz="-1.51745387499321E-07"
+        iyy="6.94753945949236E-05"
+        iyz="3.35003193615963E-07"
+        izz="2.79104313007998E-05" />
     </inertial>
     <visual>
@@ -627,5 +627,5 @@
         name="">
         <color
-          rgba="0.75294 0.75294 0.75294 1" />
+          rgba="0.752941176470588 0.752941176470588 0.752941176470588 1" />
       </material>
     </visual>
@@ -660,5 +660,5 @@
         rpy="0 0 0" />
       <mass
-        value="0.1" />
+        value="0" />
       <inertia
         ixx="0"

Commit message: adding lidar link

File: description/robot.urdf.xacro (robot description, xacro)
@@ -2,4 +2,5 @@
 <robot xmlns:xacro="http://www.ros.org/wiki/xacro" name="auriga" >
     <xacro:include filename="robot_core.xacro" />
-    <!-- <xacro:include filename="gazebo_control.xacro" /> -->
+    <xacro:include filename="gazebo_control.xacro" />
+    <xacro:include filename="lidar.xacro" />
 </robot>

File: description/robot_core.xacro (robot description, xacro)
@@ -14,25 +14,26 @@
     </material>
     <!-- The Solidworks generated urdf starts from here -->
-    <link name="dummy">
-   </link>
-    <joint name="dummy_joint" type="fixed">
-     <parent link="dummy"/>
-     <child link="base_link"/>
-   </joint>
+  <link name="dummy">
+  </link>
+  <joint name="dummy_joint" type="fixed">
+    <parent link="dummy"/>
+    <child link="base_link"/>
+  </joint>
+  <!-- <mesh filename="file://$(find auriga)/description/meshes/rocker_2_link.STL" /> -->
  <link
     name="base_link">
     <inertial>
       <origin
-        xyz="-0.13058 -0.075146 -0.064102"
-        rpy="0 0 0" />
-      <mass
-        value="7.2522" />
-      <inertia
-        ixx="0.049215"
-        ixy="1.0185E-06"
-        ixz="-5.3255E-05"
-        iyy="0.077749"
-        iyz="-0.003306"
-        izz="0.054205" />
+        xyz="-0.064102 0.13058 0.075146"
+        rpy="0 0 0" />
+      <mass
+        value="7" />
+      <inertia
+        ixx="0.054205"
+        ixy="5.3255E-05"
+        ixz="0.003306"
+        iyy="0.049215"
+        iyz="1.0185E-06"
+        izz="0.077749" />
     </inertial>
     <visual>
@@ -64,15 +65,15 @@
     <inertial>
       <origin
-        xyz="-0.00319427397416952 0.0774063348676216 0.0514223730363776"
-        rpy="0 0 0" />
-      <mass
-        value="0.157115010617485" />
-      <inertia
-        ixx="0.0029864627992537"
-        ixy="1.12349826817264E-05"
-        ixz="3.1664433625397E-05"
-        iyy="0.00259908313149434"
-        iyz="-0.000678181482698449"
-        izz="0.000411909267858246" />
+        xyz="-0.076932 -0.010223 -0.086892"
+        rpy="0 0 0" />
+      <mass
+        value="1.5" />
+      <inertia
+        ixx="0.00055446"
+        ixy="-0.00019575"
+        ixz="-0.00089962"
+        iyy="0.0036801"
+        iyz="-7.225E-05"
+        izz="0.0032548" />
     </inertial>
     <visual>
@@ -87,5 +88,5 @@
         name="">
         <color
-          rgba="0.427450980392157 0.447058823529412 0.427450980392157 1" />
+          rgba="0.42745 0.44706 0.42745 1" />
       </material>
     </visual>
@@ -104,6 +105,6 @@
     type="fixed">
     <origin
-      xyz="0.03499 -0.092655 -0.033"
-      rpy="3.1416 0 3.1416" />
+      xyz="-0.033 -0.0349903674977046 0.0926549569145568"
+      rpy="0 0 0" />
     <parent
       link="base_link" />
@@ -117,15 +118,15 @@
     <inertial>
       <origin
-        xyz="0.0023959 -0.061899 -0.00023965"
-        rpy="0 0 0" />
-      <mass
-        value="0.109" />
-      <inertia
-        ixx="0.00075509"
-        ixy="4.3842E-06"
-        ixz="1.6974E-08"
-        iyy="0.00066525"
-        iyz="2.1776E-06"
-        izz="0.00010281" />
+        xyz="-0.00063117 -0.014617 -0.067982"
+        rpy="0 0 0" />
+      <mass
+        value="1.3" />
+      <inertia
+        ixx="0.00018539"
+        ixy="-2.4832E-07"
+        ixz="9.7781E-06"
+        iyy="0.0012984"
+        iyz="-2.6746E-05"
+        izz="0.0012385" />
     </inertial>
     <visual>
@@ -157,6 +158,6 @@
     type="revolute">
     <origin
-      xyz="-0.02051 0.053967 -0.099947"
-      rpy="0 0 3.1416" />
+      xyz="0.10013 -0.02051 -0.053968"
+      rpy="0 0 0" />
     <parent
       link="rocker_1_link" />
@@ -164,5 +165,5 @@
       link="bogie_1_link" />
     <axis
-      xyz="-1 0 0" />
+      xyz="0 1 0" />
     <limit
       lower="-0.785"
@@ -175,15 +176,15 @@
     <inertial>
       <origin
-        xyz="0.00416147173779097 -9.28831021262955E-08 1.94176211321812E-07"
-        rpy="0 0 0" />
-      <mass
-        value="0.926156136524473" />
-      <inertia
-        ixx="0.00219829054546711"
-        ixy="-1.07358910102717E-08"
-        ixz="8.07356099787813E-09"
-        iyy="0.00140016164031924"
-        iyz="3.89529542945175E-08"
-        izz="0.00140018200801187" />
+        xyz="-2.0878E-07 0.0041615 5.2366E-08"
+        rpy="0 0 0" />
+      <mass
+        value="1" />
+      <inertia
+        ixx="0.0014002"
+        ixy="-1.0049E-08"
+        ixz="3.9839E-08"
+        iyy="0.0021983"
+        iyz="8.9136E-09"
+        izz="0.0014002" />
     </inertial>
     <visual>
@@ -198,5 +199,5 @@
         name="">
         <color
-          rgba="0.752941176470588 0.752941176470588 0.752941176470588 1" />
+          rgba="0.75294 0.75294 0.75294 1" />
       </material>
     </visual>
@@ -215,6 +216,6 @@
     type="continuous">
     <origin
-      xyz="0.10265 -0.079036 0.089695"
-      rpy="0 0 3.1416" />
+      xyz="-0.090727 -0.10265 -0.077849"
+      rpy="0 0 0" />
     <parent
       link="bogie_1_link" />
@@ -222,5 +223,5 @@
       link="wheel_5_link" />
     <axis
-      xyz="-1 0 0" />
+      xyz="0 1 0" />
   </joint>
   <link
@@ -228,14 +229,14 @@
     <inertial>
       <origin
-        xyz="0.0041615 -0.00034885 -0.39025"
-        rpy="0 0 0" />
-      <mass
-        value="0.92616" />
-      <inertia
-        ixx="0.0021983"
-        ixy="9.9644E-09"
-        ixz="-9.0085E-09"
-        iyy="0.0014002"
-        iyz="4.0148E-08"
+        xyz="0.38939 -0.010839 -0.00083276"
+        rpy="0 0 0" />
+      <mass
+        value="1" />
+      <inertia
+        ixx="0.0014001"
+        ixy="-1.1975E-08"
+        ixz="3.1911E-08"
+        iyy="0.0021983"
+        iyz="6.0868E-09"
         izz="0.0014002" />
     </inertial>
@@ -268,6 +269,6 @@
     type="continuous">
     <origin
-      xyz="0.10265 -0.078688 0.29995"
-      rpy="0 0 3.1416" />
+      xyz="-0.30013 -0.08765 -0.078687"
+      rpy="0 0 0" />
     <parent
       link="bogie_1_link" />
@@ -275,5 +276,5 @@
       link="wheel_6_link" />
     <axis
-      xyz="-1 0 0" />
+      xyz="0 1 0" />
   </joint>
   <link
@@ -281,15 +282,15 @@
     <inertial>
       <origin
-        xyz="0.00416147173779091 0.000348722601230034 0.39025104440836"
-        rpy="0 0 0" />
-      <mass
-        value="0.926156136524472" />
-      <inertia
-        ixx="0.00219829054546711"
-        ixy="-1.32650632923669E-08"
-        ixz="-2.11656297334914E-09"
-        iyy="0.00140013325413858"
-        iyz="-1.15497356200624E-08"
-        izz="0.00140021039419254" />
+        xyz="-0.38939 0.019161 0.00083282"
+        rpy="0 0 0" />
+      <mass
+        value="1" />
+      <inertia
+        ixx="0.0014001"
+        ixy="1.3224E-08"
+        ixz="1.2945E-08"
+        iyy="0.0021983"
+        iyz="-2.3574E-09"
+        izz="0.0014002" />
     </inertial>
     <visual>
@@ -304,5 +305,5 @@
         name="">
         <color
-          rgba="0.752941176470588 0.752941176470588 0.752941176470588 1" />
+          rgba="0.75294 0.75294 0.75294 1" />
       </material>
     </visual>
@@ -321,5 +322,5 @@
     type="continuous">
     <origin
-      xyz="-0.12316 0.13231 -0.19025"
+      xyz="0.18939 -0.12316 -0.13349"
       rpy="0 0 0" />
     <parent
@@ -328,5 +329,5 @@
       link="wheel_4_link" />
     <axis
-      xyz="-1 0 0" />
+      xyz="0 1 0" />
   </joint>
   <link
@@ -334,15 +335,15 @@
     <inertial>
       <origin
-        xyz="-0.30934 -0.015249 -0.084422"
-        rpy="0 0 0" />
-      <mass
-        value="0.15712" />
-      <inertia
-        ixx="0.0029865"
-        ixy="1.1235E-05"
-        ixz="-3.1664E-05"
-        iyy="0.0025991"
-        iyz="0.00067818"
-        izz="0.00041191" />
+        xyz="-0.10993 0.31637 0.0057628"
+        rpy="0 0 0" />
+      <mass
+        value="1.5" />
+      <inertia
+        ixx="0.00055446"
+        ixy="0.00019575"
+        ixz="-0.00089962"
+        iyy="0.0036801"
+        iyz="7.225E-05"
+        izz="0.0032548" />
     </inertial>
     <visual>
@@ -387,15 +388,15 @@
     <inertial>
       <origin
-        xyz="0.00239591308301151 0.0617953988436242 0.00358741675136703"
-        rpy="0 0 0" />
-      <mass
-        value="0.108995977851336" />
-      <inertia
-        ixx="0.0007550940265459"
-        ixy="-4.37688335423889E-06"
-        ixz="-2.54091808736551E-07"
-        iyy="0.000663370668469634"
-        iyz="3.25430149906427E-05"
-        izz="0.000104686998401709" />
+        xyz="-0.00022018 0.014617 -0.067984"
+        rpy="0 0 0" />
+      <mass
+        value="1.3" />
+      <inertia
+        ixx="0.00018531"
+        ixy="8.6623E-08"
+        ixz="3.4111E-06"
+        iyy="0.0012984"
+        iyz="2.6747E-05"
+        izz="0.0012386" />
     </inertial>
     <visual>
@@ -410,5 +411,5 @@
         name="">
         <color
-          rgba="0.427450980392157 0.447058823529412 0.427450980392157 1" />
+          rgba="0.42745 0.44706 0.42745 1" />
       </material>
     </visual>
@@ -427,6 +428,6 @@
     type="revolute">
     <origin
-      xyz="-0.32665 -0.038665 0.067793"
-      rpy="3.1416 0 3.1416" />
+      xyz="0.0670443300803985 0.326654617315038 0.0386879525429506"
+      rpy="0 0 0" />
     <parent
       link="rocker_2_link" />
@@ -434,5 +435,5 @@
       link="bogie_2_link" />
     <axis
-      xyz="-1 0 0" />
+      xyz="0 -1 0" />
     <limit
       lower="-0.785"
@@ -445,15 +446,15 @@
     <inertial>
       <origin
-        xyz="-2.1518E-07 -5.3832E-09 -0.0041615"
-        rpy="0 0 0" />
-      <mass
-        value="0.92616" />
-      <inertia
-        ixx="0.0014001"
-        ixy="3.1138E-08"
-        ixz="1.2067E-08"
-        iyy="0.0014002"
-        iyz="-5.9011E-09"
-        izz="0.0021983" />
+        xyz="1.1827E-07 -0.0041615 1.7985E-07"
+        rpy="0 0 0" />
+      <mass
+        value="1" />
+      <inertia
+        ixx="0.0014002"
+        ixy="-1.366E-09"
+        ixz="-9.1487E-09"
+        iyy="0.0021983"
+        iyz="-1.3363E-08"
+        izz="0.0014001" />
     </inertial>
     <visual>
@@ -485,6 +486,6 @@
     type="continuous">
     <origin
-      xyz="0.10265 0.07334 0.094409"
-      rpy="0 1.5708 0" />
+      xyz="-0.090254 0.10265 -0.078396"
+      rpy="0 0 0" />
     <parent
       link="bogie_2_link" />
@@ -492,5 +493,5 @@
       link="wheel_2_link" />
     <axis
-      xyz="0 0 1" />
+      xyz="0 -1 0" />
   </joint>
   <link
@@ -498,14 +499,14 @@
     <inertial>
       <origin
-        xyz="-0.0041615 -2.0875E-07 5.2503E-08"
-        rpy="0 0 0" />
-      <mass
-        value="0.92616" />
-      <inertia
-        ixx="0.0021983"
-        ixy="1.0043E-08"
-        ixz="-8.9202E-09"
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